File: usb-c-pd-supply.kicad_pcb (KiCad board)
At the start: 4 copper layers, 60 x 40 mm, 41 parts, among them J1 USB_C_Receptacle_USB2.0_14P, J2 Output connector, Q1 2N7002E, Q2 IRLML6401, SW1 Voltage selector, U1 TPS70933DBVR, U2 CH224K, U3 MC14051BDR2G

Commit message: Add files via upload
Parts:
- added D10: Green, LED_SMD:LED_0805_2012Metric, F.Cu at (115.5, 123.8)
- added R13: 1K, Resistor_SMD:R_0805_2012Metric, F.Cu at (115.6, 121.5)
- D3: value LED1 -> Red
- D4: value LED2 -> Green
- D5: value LED3 -> Green
- D6: value LED4 -> Green
- D7: value LED5 -> Green
- Q2: value IRLML6401 -> DMN3404L-7
- moved R6 3.81 mm to (119.3, 121.5)
- moved D4 3.81 mm to (119.2, 123.8)
- moved R12 0.74 mm to (119.3, 101.0)
Connections:
- R6 pad 1: Net-(U3-X3) -> Net-(U3-X2)
- U3 pad 15: unconnected-(U3-X2-Pad15) -> Net-(U3-X2)
Routing:
- net Net-(U3-X2): track 0.00 -> 9.96 mm
- net GND: track 68.0 -> 73.5 mm
- net Net-(D10-A): track 0.00 -> 2.33 mm
- net Net-(D9-A): track 6.16 -> 5.43 mm
Other:
- board text added: "15V"

Commit message: Add files via upload
Parts:
- renumbered C4 to C3, C5 to C4, C6 to C5, C7 to C6, C9 to C7, D8 to D1, D7 to D10, D1 to D2, D2 to D3, D3 to D4, D9 to D5, D4 to D6, D10 to D7, D5 to D8, D6 to D9, R10 to R1, R13 to R10, R7 to R11, R8 to R12, R9 to R13, R11 to R2, R1 to R3, R2 to R4, R3 to R5, R4 to R6, R5 to R7, R12 to R8, R6 to R9
