File: usb-c-pd-supply.kicad_sch (KiCad schematic)
At the start: 41 parts, among them J1 USB_C_Receptacle_USB2.0_14P, J2 Output connector, Q1 2N7002E, Q2 DMN3404L-7, SW1 Voltage selector, U1 TPS70933DBVR, U2 CH224K, U3 MC14051BDR2G

Commit message: Add files via upload
Parts:
- added D10: Green, LED_SMD:LED_0805_2012Metric, symbol Device:LED
- added R13: 1K, Resistor_SMD:R_0805_2012Metric, symbol Device:R
Connections:
- net GND: now also D10.1 (K)
- net at R6.1: now also U3.15 (X2); no longer U3.12 (X3)
- new net: R13.1, U3.12 (X3)
- new net: D10.2 (A), R13.2
- no-connect marks 1 -> 0
Other:
- note added: "15V"
- moved on the sheet: D4, D5, D6, D7, R6, R7, R8, R9

Commit message: Add files via upload
Parts:
- renumbered C4 to C3, C5 to C4, C6 to C5, C7 to C6, C9 to C7, D8 to D1, D7 to D10, D1 to D2, D2 to D3, D3 to D4, D9 to D5, D4 to D6, D10 to D7, D5 to D8, D6 to D9, R10 to R1, R13 to R10, R7 to R11, R8 to R12, R9 to R13, R11 to R2, R1 to R3, R2 to R4, R3 to R5, R4 to R6, R5 to R7, R12 to R8, R6 to R9
